File: Hardware/XBee_Explorer Thin.sch (EAGLE design)
At the start: 50 parts, among them J4 QWIIC_RIGHT_ANGLE, Q1 3.1A/30V/105mΩ, U1 FSUSB30MUX_MSOP10, U2 MCP73831, U4 CP210X, U5 AP7361C-33

Commit message: Adds higher current capable switching regulator
Parts:
- removed C11: 4.7uF, SparkFun-Capacitors:4.7UF-0603-6.3V-(10%)
- removed Q1: 3.1A/30V/105mΩ, SparkFun-DiscreteSemi:MOSFET_PCH-DMG2307L
- removed R9: 100k, SparkFun-Resistors:100KOHM-0603-1/10W-1%
- removed U5: AP7361C-33, SparkFun-IC-Power:AP7361C-33FGEUDFN-8
- added C1, C10: 22uF, SparkFun-Capacitors:22UF-1210-16V-20%
- added C15: 0.22uF, SparkFun-Capacitors:0.22UF-0603-50V-10%
- added C2: 1.0uF, SparkFun-Capacitors:1.0UF-0603-16V-10%
- added C9: 0.1uF, SparkFun-Capacitors:0.1UF-0603-100V-10%
- added D6: 3A/40V/500mV, SparkFun-DiscreteSemi:DIODE-SCHOTTKY-B340A
- added L2: 2.2uH, SparkFun-Coils:2.2μH_SHIELDED_INDUCTOR_5X5
- added Q2: 3.1A/30V/105mΩ, SparkFun-DiscreteSemi:MOSFET_PCH-DMG2307L
- added R17, R19: 100k, SparkFun-Resistors:100KOHM-0603-1/10W-1%
- added R18: 43k, SparkFun-Resistors:43KOHM-0603-1/10W-1%
- added R20: 10k, SparkFun-Resistors:10KOHM-0603-1/10W-1%
- added S4: (no value), SparkFun-Switches:SWITCH-SPDT-SMD-AYZ0202
- added U6: LMR33630, SparkFun-IC-Power:LMR33630
- C5: value 4.7uF -> 10uF; device SparkFun-Capacitors:4.7UF-0603-6.3V-(10%) -> SparkFun-Capacitors:10UF-0603-6.3V-20%
- D1: value 3.3V -> 3A/10V/280mV; device SparkFun-DiscreteSemi:DIODE-ZENER-MM3Z3V3T1G -> SparkFun-DiscreteSemi:DIODE-SCHOTTKY-BAT60A
- D5: value 3A/40V/500mV -> 3A/10V/280mV; device SparkFun-DiscreteSemi:DIODE-SCHOTTKY-B340A -> SparkFun-DiscreteSemi:DIODE-SCHOTTKY-BAT60A
- R6: value 10k -> 100k; device SparkFun-Resistors:10KOHM-0603-1/10W-1% -> SparkFun-Resistors:100KOHM-0603-1/10W-1%
Connections:
- removed net 3.3V_EN_VE: D1.C, R9.1, U5.EN
- removed net N$25: JP2.!CS!/!CTS2!/DIO3
- removed net N$26: JP2.PICO/TX2/DIO4
- removed net N$27: JP2.ASSOCIATE/DIO5
- removed net N$28: JP2.!RTS!/DIO6
- removed net N$29: JP2.!CTS!/DIO7
- removed net N$30: JP2.DTR/DIO8
- removed net N$31: JP2.!SLEEP!/DIO9
- removed net N$32: JP2.POCI/DIO12
- removed net N$35: U1.!OE!
- removed net VCC: C5.1, D5.C, Q1.S, R9.2, U5.IN
- new net DIRECT_SELECT: S4.P, U1.S
- new net N$17: C9.1, U6.BOOT
- new net N$18: R17.1, R18.2, U6.FB
- new net N$19: R19.1, U6.PGOOD
- new net N$20: C2.1, R19.2, U6.VCC
- new net N$22: R6.2, S4.S
- new net SW: C9.2, L2.1, U6.NC, U6.SW
- new net VIN: D1.C, D5.C, D6.A, Q2.G, R1.2, R20.2, U4.VREGIN
- new net V_USB_2: D1.A, J1.VBUS
- net 3.3V: now also C1.1, C10.1, L2.2, R17.2, R6.1; no longer C11.1, U5.OUT
- net D10/RSSI_PWM: now also JP2.VUSB/RSSI/DIO10
- net D12/SPI_MISO: now also JP2.POCI/DIO12
- net D3/!CS!: now also JP2.!CS!/!CTS2!/DIO3
- net D4/SPI_MOSI: now also JP2.PICO/TX2/DIO4
- net D5/ASSOCIATE: now also JP2.ASSOCIATE/DIO5
- net D6/!RTS!: now also JP2.!RTS!/DIO6
- net D7/!CTS!: now also JP2.!CTS!/DIO7
- net D8/!DTR!: now also JP2.DTR/DIO8
- net D9/!SLEEP!: now also JP2.!SLEEP!/DIO9
- net GND: now also C1.2, C10.2, C15.2, C2.2, R18.1, R20.1, S4.O, U1.!OE!, U6.AGND, U6.PGND; no longer C11.2, D1.A, R6.1, U5.GND
- net N$15: now also C15.1, C5.1, D6.C, Q2.S, U6.EN, U6.VIN; no longer JP2.VUSB/RSSI/DIO10
- net V_BATT: now also Q2.D; no longer Q1.D
- net V_USB: no longer J1.VBUS, Q1.G, R1.2, R6.2, U4.VREGIN
Other:
- note added: "Charge Rate: 500mA"
- note added: "Default (Low) = SDA (I2C)"
- note removed: "235mA peak"
- note removed: "Input: 3.7-6.0V Output: 1A Max"
- note removed: "Might not need 1.0uF for modules with headers"
- note removed: "Output: 500mA"
- note removed: "PTH"
- moved on the sheet: C3, C4, C5, C6, C7, D4, D5, J1, J12, J3, J8, JP2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

Commit message: Using new VREG, adds documentation for new VREG
Parts:
- removed C10: 22uF, SparkFun-Capacitors:22UF-1210-16V-20%
- removed C15: 0.22uF, SparkFun-Capacitors:0.22UF-0603-50V-10%
- removed C5: 10uF, SparkFun-Capacitors:10UF-0603-6.3V-20%
- removed C9: 0.1uF, SparkFun-Capacitors:0.1UF-0603-100V-10%
- removed D4: Yellow, SparkFun-LED:LED-YELLOW0603
- removed L2: 2.2uH, SparkFun-Coils:2.2μH_SHIELDED_INDUCTOR_5X5
- removed R17, R19: 100k, SparkFun-Resistors:100KOHM-0603-1/10W-1%
- removed R18: 43k, SparkFun-Resistors:43KOHM-0603-1/10W-1%
- removed U6: LMR33630, SparkFun-IC-Power:LMR33630
- added JP1, JP3: JUMPER-SMT_2_NC_TRACE_SILK, SparkFun-Jumpers:JUMPER-SMT_2_NC_TRACE_SILK
- added L1: 4.7μH, SparkFun-Coils:4.7μH_SHIELDED_INDUCTORNPIS_LS
- added LOGO1: SFE_LOGO_NAME_FLAME.1_INCH, SparkFun-Aesthetics:SFE_LOGO_NAME_FLAME.1_INCH
- added LOGO2: OSHW-LOGOS, SparkFun-Aesthetics:OSHW-LOGOS
- added LOGO3: QWIIC_LOGO_3MM, SparkFun-Aesthetics:QWIIC_LOGO_3MM
- C1: value 22uF -> 10uF; device SparkFun-Capacitors:22UF-1210-16V-20% -> SparkFun-Capacitors:10UF-1210-50V-20%
- C2: value 1.0uF -> 0.1uF; device SparkFun-Capacitors:1.0UF-0603-16V-10% -> SparkFun-Capacitors:0.1UF-0603-25V-5%
- C3: value 4.7uF -> 22uF; device SparkFun-Capacitors:4.7UF-0603-6.3V-(10%) -> SparkFun-Capacitors:22UF-0603-6.3V-20%
- C4: value 4.7uF -> 22uF; device SparkFun-Capacitors:4.7UF-0603-35V-(20%) -> SparkFun-Capacitors:22UF-0603-6.3V-20%
- R3: value 4.7k -> 100k; device SparkFun-Resistors:4.7KOHM-0603-1/10W-1% -> SparkFun-Resistors:100KOHM-0603-1/10W-1%
- R4: value 2.0k -> 100k; device SparkFun-Resistors:2.0KOHM-0603-1/10W-5% -> SparkFun-Resistors:100KOHM-0603-1/10W-1%
- U2: value MCP73831 -> AP63203; device SparkFun-IC-Power:MCP73831 -> SparkFun-IC-Power:AP63203
Connections:
- removed net N$10: C3.1, R3.1, U2.VIN
- removed net N$17: C9.1, U6.BOOT
- removed net N$18: R17.1, R18.2, U6.FB
- removed net N$19: R19.1, U6.PGOOD
- removed net N$20: C2.1, R19.2, U6.VCC
- removed net N$9: D4.A, R3.2
- removed net SDA: U1.D1+
- removed net SW: C9.2, L2.1, U6.NC, U6.SW
- new net EN: J5.7, R3.1, R4.2, U2.EN
- new net N$21: D3.C, JP3.2
- new net N$23: D2.C, JP1.2
- net 3.3V: now also C3.1, C4.1, L1.2, U2.FB; no longer C1.1, C10.1, L2.2, R17.2
- net D11/SDA: now also U1.D1+
- net GND: now also JP1.1, JP3.1, U2.GND; no longer C10.2, C15.2, C2.2, C5.2, D2.C, D3.C, R18.1, U2.VSS, U6.AGND, U6.PGND
- net N$1: now also C2.1, U2.BST; no longer R4.2, U2.PROG
- net N$15: now also C1.1, R3.2, U2.VIN; no longer C15.1, C5.1, U6.EN, U6.VIN
- net N$8: now also C2.2, L1.1, U2.SW; no longer D4.C, U2.STAT
- net V_BATT: no longer C4.1, U2.VBAT
Other:
- note added: "Buck Converter - AP63203"
- note added: "Buttons and LEDs"
- note added: "Default (Low) = I2C (SDA)"
- note added: "Lipo Battery Connector"
- note added: "USB Switch - FSUSB30"
- note added: "VIN: 3.8 - 32V Iout: 2A Max"
- note removed: "Charge Rate: 500mA"
- note removed: "Lipo Battery Charger"
- note removed: "Need jumpers here"
- note removed: "Voltage Regulation"
- moved on the sheet: C1, C2, C3, C4, D2, D3, D6, I2C_PU, J12, J4, J5, J6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

Commit message: Updates schematic
Parts:
- removed R10: 33k, SparkFun-Resistors:33KOHM-0603-1/10W-1%
- removed R2, R5: 4.7k, SparkFun-Resistors:4.7KOHM-0603-1/10W-1%
- removed R6: 100k, SparkFun-Resistors:100KOHM-0603-1/10W-1%
- removed S4: (no value), SparkFun-Switches:SWITCH-SPDT-SMD-AYZ0202
- removed U4: CP210X, SparkFun-IC-Comms:CP2102N
- added C10: 10uF, SparkFun-Capacitors:10UF-0603-6.3V-20%
- added C5, C9: 0.1uF, SparkFun-Capacitors:0.1UF-0603-25V-(+80/-20%)
- added C8: 4.7uF, SparkFun-Capacitors:4.7UF-0603-6.3V-(10%)
- added H1, H2, H3, H4: STAND-OFFTIGHT, SparkFun-Hardware:STAND-OFFTIGHT
- added R17: 22k, SparkFun-Resistors:22KOHM-0402_TIGHT-1/10W-1%
- added R18: 33k, SparkFun-Resistors:33KOHM-0402T-1/16W-1%
- added R9: 10k, SparkFun-Resistors:10KOHM-0402T-1/16W-1%
- added S3: (no value), SparkFun-Switches:SWITCH-DPDT-SMD-AYZ0202
- added U3, U5: ESD Diode, SparkFun-DiscreteSemi:TVS_DIODE_ARRAY_DT1042-04SO-7
- added U6: CP210X, SparkFun-IC-Comms:CP2102N
- C6: value 0.1uF -> 10nF; device SparkFun-Capacitors:0.1UF-0603-25V-(+80/-20%) -> SparkFun-Capacitors:10NF-0603-50V-10%
- C7: value 4.7uF -> 10nF; device SparkFun-Capacitors:4.7UF-0603-6.3V-(10%) -> SparkFun-Capacitors:10NF-0603-50V-10%
- R1: value 22k -> 100k; device SparkFun-Resistors:22KOHM-0603-1/10W-1% -> SparkFun-Resistors:100KOHM-0603-1/10W-1%
- R11: value 2.2k -> 1k; device SparkFun-Resistors:2.2KOHM-0603-1/10W-1% -> SparkFun-Resistors:1KOHM-0603-1/10W-1%
Connections:
- removed net D12/SPI_MISO: J6.4, JP2.POCI/DIO12
- removed net D3/!CS!: J5.4, JP2.!CS!/!CTS2!/DIO3
- removed net D4/SPI_MOSI: J5.10, JP2.PICO/TX2/DIO4
- removed net N$2: R1.1, R10.2, U4.VBUS
- removed net N$22: R6.2, S4.S
- removed net N$6: R2.2, U4.!RSTB
- new net D12/SPI_POCI: J5.5, JP2.POCI/DIO12
- new net D3/SPI_!CS!: J5.3, JP2.!CS!/!CTS2!/DIO3/AD3
- new net D4/SPI_PICO: J5.4, JP2.PICO/TX2/DIO4
- new net GND1: C5.2
- new net N$10: R17.1, R18.2, U6.VBUS
- new net N$9: R9.2, U6.!RSTB
- net !RESET!: now also C6.1, J6.4; no longer J6.5, R5.1
- net 3.3V: now also C10.1, C5.1, C7.1, C8.1, C9.1, J6.9, R1.1, R9.1, U6.VDD, U6.VIO, U6.VREGIN; no longer J6.1, R5.2, R6.1
- net D+: now also U5.IO4, U6.D+; no longer U4.D+
- net D-: now also U5.IO3, U6.D-; no longer U4.D-
- net D0: now also JP2.DIO0/AD0; no longer JP2.DIO0
- net D1/SCL: now also J6.7, JP2.SCL/DIO1/AD1; no longer J5.2, JP2.SCL/DIO1
- net D10/RSSI_PWM: now also J6.5; no longer J6.6
- net D11/SDA: now also J6.8; no longer J6.7
- net D13/TXO: now also J6.1, U6.RXD; no longer J6.2, U4.RXD
- net D14/RXI: now also J6.2, U6.TXD; no longer J6.3, U4.TXD
- net D2/SPI_CLK: now also J5.2, JP2.ATTN/CLK/!RTS2!/DIO2/AD2; no longer J5.3, JP2.ATTN/CLK/!RTS2!/DIO2
- net D5/ASSOCIATE: now also J5.7; no longer J5.6
- net D6/!RTS!: now also J5.6, U6.RTS; no longer J5.5, U4.RTS
- net D7/!CTS!: now also J5.10; no longer J5.9
- net D8/!DTR!: now also J5.8, U6.DTR; no longer J6.9, U4.DTR
- net D9/!SLEEP!: now also J5.9; no longer J5.8
- net DIRECT_D+: now also U3.IO4
- net DIRECT_D-: now also U3.IO3
- net DIRECT_SELECT: now also S3.2, S3.5; no longer S4.P
- net EN: now also J6.6; no longer J5.7
- net GND: now also C10.2, C8.2, C9.2, R18.1, S3.1, S3.3, U3.VSS, U5.VSS, U6.GND; no longer R10.1, S4.O, U4.GND
- net N$3: now also R1.2, S3.4, S3.6; no longer C6.1, C7.1, R2.1, U4.VDD, U4.VIO
- net VIN: now also R17.2; no longer R1.2, U4.VREGIN
- net V_USB: now also U5.VCC
- net V_USB_2: now also U3.VCC
Other:
- note added: "USB-C Connectors"
- moved on the sheet: C1, C2, C3, C4, C6, C7, D1, D5, D6, J1, J3, JP2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

Commit message: General placement of parts within the board
Connections:
- removed net GND1: C5.2
- net D13/TXO: now also J6.2; no longer J6.1
- net D14/RXI: now also J6.3; no longer J6.2
- net D5/ASSOCIATE: now also J5.6; no longer J5.7
- net D6/!RTS!: now also J5.7; no longer J5.6
- net D7/!CTS!: now also J5.8; no longer J5.10
- net D8/!DTR!: now also J5.9; no longer J5.8
- net D9/!SLEEP!: now also J5.10; no longer J5.9
- net GND: now also C5.2
- net VIN: now also J6.1
Other:
- moved on the sheet: R17, R18

Commit message: Routes some airwires
Parts:
- R17: device SparkFun-Resistors:22KOHM-0402_TIGHT-1/10W-1% -> SparkFun-Resistors:22KOHM-0603-1/10W-1%
- R18: device SparkFun-Resistors:33KOHM-0402T-1/16W-1% -> SparkFun-Resistors:33KOHM-0603-1/10W-1%
- R9: device SparkFun-Resistors:10KOHM-0402T-1/16W-1% -> SparkFun-Resistors:10KOHM-0603-1/10W-1%
Connections:
- net GND: now also S3.6; no longer S3.1
- net N$3: now also S3.1; no longer S3.6
Changed lines of the file:
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@@
 <part name="JP2" library="xbee_improved" deviceset="XBEE_UPDATE" device="XBEE_SMD"/>
 <part name="U6" library="SparkFun-IC-Comms" deviceset="CP2102N" device="" value="CP210X"/>
-<part name="R9" library="SparkFun-Resistors" deviceset="10KOHM" device="-0402T-1/16W-1%" value="10k"/>
+<part name="R9" library="SparkFun-Resistors" deviceset="10KOHM" device="-0603-1/10W-1%" value="10k"/>
 <part name="SUPPLY22" library="SparkFun-PowerSymbols" deviceset="3.3V" device=""/>
 <part name="GND30" library="SparkFun-PowerSymbols" deviceset="GND" device=""/>
-<part name="R17" library="SparkFun-Resistors" deviceset="22KOHM" device="-0402_TIGHT-1/10W-1%" value="22k"/>
-<part name="R18" library="SparkFun-Resistors" deviceset="33KOHM" device="-0402T-1/16W-1%" value="33k"/>
+<part name="R17" library="SparkFun-Resistors" deviceset="22KOHM" device="-0603-1/10W-1%" value="22k"/>
+<part name="R18" library="SparkFun-Resistors" deviceset="33KOHM" device="-0603-1/10W-1%" value="33k"/>
 <part name="GND32" library="SparkFun-PowerSymbols" deviceset="GND" device=""/>
 <part name="SUPPLY21" library="SparkFun-PowerSymbols" deviceset="VIN" device=""/>
@@
 </segment>
 <segment>
-<pinref part="S3" gate="G$1" pin="1"/>
-<wire x1="17.78" y1="55.88" x2="20.32" y2="55.88" width="0.1524" layer="91"/>
-<wire x1="17.78" y1="55.88" x2="17.78" y2="50.8" width="0.1524" layer="91"/>
+<wire x1="17.78" y1="58.42" x2="17.78" y2="50.8" width="0.1524" layer="91"/>
 <pinref part="S3" gate="G$1" pin="3"/>
 <wire x1="17.78" y1="50.8" x2="17.78" y2="43.18" width="0.1524" layer="91"/>
@@
 <junction x="17.78" y="50.8"/>
 <pinref part="GND36" gate="1" pin="GND"/>
+<pinref part="S3" gate="G$1" pin="6"/>
+<wire x1="20.32" y1="58.42" x2="17.78" y2="58.42" width="0.1524" layer="91"/>
 </segment>
 <segment>
@@
 <net name="N$3" class="0">
 <segment>
-<pinref part="S3" gate="G$1" pin="6"/>
-<wire x1="20.32" y1="58.42" x2="17.78" y2="58.42" width="0.1524" layer="91"/>
 <wire x1="20.32" y1="63.5" x2="17.78" y2="63.5" width="0.1524" layer="91"/>
 <pinref part="R1" gate="G$1" pin="2"/>
 <wire x1="17.78" y1="63.5" x2="17.78" y2="66.04" width="0.1524" layer="91"/>
 <pinref part="S3" gate="G$1" pin="4"/>
-<wire x1="17.78" y1="58.42" x2="17.78" y2="63.5" width="0.1524" layer="91"/>
+<pinref part="S3" gate="G$1" pin="1"/>
+<wire x1="20.32" y1="55.88" x2="15.24" y2="55.88" width="0.1524" layer="91"/>
+<wire x1="15.24" y1="55.88" x2="15.24" y2="63.5" width="0.1524" layer="91"/>
+<wire x1="15.24" y1="63.5" x2="17.78" y2="63.5" width="0.1524" layer="91"/>
 <junction x="17.78" y="63.5"/>
 </segment>

Commit message: Removes VIN from pin one one header and puts it at pin 10
* Shifts all other nets up one to accommodate VIN
Connections:
- net !RESET!: now also J6.3; no longer J6.4
- net 3.3V: now also J6.8; no longer J6.9
- net D1/SCL: now also J6.6; no longer J6.7
- net D10/RSSI_PWM: now also J6.4; no longer J6.5
- net D11/SDA: now also J6.7; no longer J6.8
- net D13/TXO: now also J6.1; no longer J6.2
- net D14/RXI: now also J6.2; no longer J6.3
- net EN: now also J6.5; no longer J6.6
- net GND: now also J6.9; no longer J6.10
- net VIN: now also J6.10; no longer J6.1
Changed lines of the file:
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@@
 <part name="J6" library="SparkFun-Connectors" deviceset="CONN_10" device="NO_SILK_PTH_FEMALE"/>
 <part name="SUPPLY6" library="SparkFun-PowerSymbols" deviceset="3.3V" device=""/>
-<part name="GND18" library="SparkFun-PowerSymbols" deviceset="GND" device=""/>
 <part name="R11" library="SparkFun-Resistors" deviceset="1KOHM" device="-0603-1/10W-1%" value="1k"/>
 <part name="D2" library="SparkFun-LED" deviceset="LED-RED" device="0603" value="RED"/>
@@
 <part name="SUPPLY14" library="SparkFun-PowerSymbols" deviceset="3.3V" device=""/>
 <part name="SUPPLY13" library="SparkFun-PowerSymbols" deviceset="VIN" device=""/>
+<part name="GND8" library="SparkFun-PowerSymbols" deviceset="GND" device=""/>
 </parts>
 <sheets>
@@
 <attribute name="NAME" x="27.94" y="134.112" size="1.778" layer="95" font="vector" rot="MR180"/>
 </instance>
-<instance part="SUPPLY6" gate="G$1" x="40.64" y="165.1" smashed="yes">
-<attribute name="VALUE" x="40.64" y="167.894" size="1.778" layer="96" font="vector" align="bottom-center"/>
-</instance>
-<instance part="GND18" gate="1" x="40.64" y="132.08" smashed="yes">
-<attribute name="VALUE" x="40.64" y="131.826" size="1.778" layer="96" font="vector" align="top-center"/>
+<instance part="SUPPLY6" gate="G$1" x="43.18" y="167.64" smashed="yes">
+<attribute name="VALUE" x="43.18" y="170.434" size="1.778" layer="96" font="vector" align="bottom-center"/>
 </instance>
 <instance part="R11" gate="G$1" x="289.56" y="68.58" smashed="yes" rot="MR270">
@@
 <attribute name="VALUE" x="17.78" y="81.534" size="1.778" layer="96" font="vector" rot="MR0" align="bottom-center"/>
 </instance>
-<instance part="SUPPLY13" gate="G$1" x="45.72" y="165.1" smashed="yes">
-<attribute name="VALUE" x="45.72" y="167.894" size="1.778" layer="96" font="vector" align="bottom-center"/>
+<instance part="SUPPLY13" gate="G$1" x="40.64" y="162.56" smashed="yes">
+<attribute name="VALUE" x="40.64" y="165.354" size="1.778" layer="96" font="vector" align="bottom-center"/>
+</instance>
+<instance part="GND8" gate="1" x="43.18" y="134.62" smashed="yes" rot="MR0">
+<attribute name="VALUE" x="43.18" y="134.366" size="1.778" layer="96" font="vector" rot="MR0" align="top-center"/>
 </instance>
 </instances>
@@
 </segment>
 <segment>
-<wire x1="43.18" y1="142.24" x2="38.1" y2="142.24" width="0.1524" layer="91"/>
-<label x="43.18" y="142.24" size="1.27" layer="95" font="vector" xref="yes"/>
-<pinref part="J6" gate="J1" pin="8"/>
+<wire x1="45.72" y1="144.78" x2="38.1" y2="144.78" width="0.1524" layer="91"/>
+<label x="45.72" y="144.78" size="1.27" layer="95" font="vector" xref="yes"/>
+<pinref part="J6" gate="J1" pin="7"/>
 </segment>
 </net>
@@
 </segment>
 <segment>
-<wire x1="43.18" y1="144.78" x2="38.1" y2="144.78" width="0.1524" layer="91"/>
-<label x="43.18" y="144.78" size="1.27" layer="95" font="vector" xref="yes"/>
-<pinref part="J6" gate="J1" pin="7"/>
+<wire x1="45.72" y1="147.32" x2="38.1" y2="147.32" width="0.1524" layer="91"/>
+<label x="45.72" y="147.32" size="1.27" layer="95" font="vector" xref="yes"/>
+<pinref part="J6" gate="J1" pin="6"/>
 </segment>
 </net>
@@
 </segment>
 <segment>
-<wire x1="40.64" y1="137.16" x2="38.1" y2="137.16" width="0.1524" layer="91"/>
-<wire x1="40.64" y1="137.16" x2="40.64" y2="134.62" width="0.1524" layer="91"/>
-<pinref part="J6" gate="J1" pin="10"/>
-<pinref part="GND18" gate="1" pin="GND"/>
-</segment>
-<segment>
 <wire x1="35.56" y1="203.2" x2="38.1" y2="203.2" width="0.1524" layer="91"/>
 <wire x1="35.56" y1="200.66" x2="35.56" y2="203.2" width="0.1524" layer="91"/>
@@
 <pinref part="GND34" gate="1" pin="GND"/>
 <wire x1="330.2" y1="223.52" x2="330.2" y2="218.44" width="0.1524" layer="91"/>
+</segment>
+<segment>
+<wire x1="43.18" y1="139.7" x2="38.1" y2="139.7" width="0.1524" layer="91"/>
+<wire x1="43.18" y1="139.7" x2="43.18" y2="137.16" width="0.1524" layer="91"/>
+<pinref part="J6" gate="J1" pin="9"/>
+<pinref part="GND8" gate="1" pin="GND"/>
 </segment>
 </net>
@@
 </segment>
 <segment>
+<wire x1="43.18" y1="142.24" x2="43.18" y2="167.64" width="0.1524" layer="91"/>
+<wire x1="38.1" y1="142.24" x2="43.18" y2="142.24" width="0.1524" layer="91"/>
+<pinref part="J6" gate="J1" pin="8"/>
 <pinref part="SUPPLY6" gate="G$1" pin="3.3V"/>
-<wire x1="40.64" y1="139.7" x2="40.64" y2="165.1" width="0.1524" layer="91"/>
-<pinref part="J6" gate="J1" pin="9"/>
-<wire x1="38.1" y1="139.7" x2="40.64" y2="139.7" width="0.1524" layer="91"/>
 </segment>
 </net>
@@
 </segment>
 <segment>
-<wire x1="43.18" y1="157.48" x2="38.1" y2="157.48" width="0.1524" layer="91"/>
-<label x="43.18" y="157.48" size="1.27" layer="95" font="vector" xref="yes"/>
-<pinref part="J6" gate="J1" pin="2"/>
+<wire x1="45.72" y1="160.02" x2="38.1" y2="160.02" width="0.1524" layer="91"/>
+<label x="45.72" y="160.02" size="1.27" layer="95" font="vector" xref="yes"/>
+<pinref part="J6" gate="J1" pin="1"/>
 </segment>
 </net>
@@
 </segment>
 <segment>
-<wire x1="43.18" y1="154.94" x2="38.1" y2="154.94" width="0.1524" layer="91"/>
-<label x="43.18" y="154.94" size="1.27" layer="95" font="vector" xref="yes"/>
-<pinref part="J6" gate="J1" pin="3"/>
+<wire x1="45.72" y1="157.48" x2="38.1" y2="157.48" width="0.1524" layer="91"/>
+<label x="45.72" y="157.48" size="1.27" layer="95" font="vector" xref="yes"/>
+<pinref part="J6" gate="J1" pin="2"/>
 </segment>
 </net>
@@
 </segment>
 <segment>
-<wire x1="43.18" y1="152.4" x2="38.1" y2="152.4" width="0.1524" layer="91"/>
-<label x="43.18" y="152.4" size="1.27" layer="95" font="vector" xref="yes"/>
-<pinref part="J6" gate="J1" pin="4"/>
+<wire x1="45.72" y1="154.94" x2="38.1" y2="154.94" width="0.1524" layer="91"/>
+<label x="45.72" y="154.94" size="1.27" layer="95" font="vector" xref="yes"/>
+<pinref part="J6" gate="J1" pin="3"/>
 </segment>
 </net>
@@
 </segment>
 <segment>
-<wire x1="43.18" y1="149.86" x2="38.1" y2="149.86" width="0.1524" layer="91"/>
-<label x="43.18" y="149.86" size="1.27" layer="95" font="vector" xref="yes"/>
-<pinref part="J6" gate="J1" pin="5"/>
+<wire x1="45.72" y1="152.4" x2="38.1" y2="152.4" width="0.1524" layer="91"/>
+<label x="45.72" y="152.4" size="1.27" layer="95" font="vector" xref="yes"/>
+<pinref part="J6" gate="J1" pin="4"/>
 </segment>
 </net>
@@
 </segment>
 <segment>
-<pinref part="J6" gate="J1" pin="1"/>
-<wire x1="38.1" y1="160.02" x2="45.72" y2="160.02" width="0.1524" layer="91"/>
-<wire x1="45.72" y1="160.02" x2="45.72" y2="165.1" width="0.1524" layer="91"/>
+<pinref part="J6" gate="J1" pin="10"/>
+<wire x1="38.1" y1="137.16" x2="40.64" y2="137.16" width="0.1524" layer="91"/>
+<wire x1="40.64" y1="137.16" x2="40.64" y2="162.56" width="0.1524" layer="91"/>
 <pinref part="SUPPLY13" gate="G$1" pin="VIN"/>
 </segment>
@@
 </segment>
 <segment>
-<pinref part="J6" gate="J1" pin="6"/>
-<wire x1="43.18" y1="147.32" x2="38.1" y2="147.32" width="0.1524" layer="91"/>
-<label x="43.18" y="147.32" size="1.27" layer="95" font="vector" xref="yes"/>
-</segment>
-</net>
+<wire x1="45.72" y1="149.86" x2="38.1" y2="149.86" width="0.1524" layer="91"/>
+<label x="45.72" y="149.86" size="1.27" layer="95" font="vector" xref="yes"/>
+<pinref part="J6" gate="J1" pin="5"/>
+</segment>
+</net>
