File: Hardware/XBee_Explorer Thin.sch (EAGLE design)
At the start: 65 parts, among them J4 QWIIC_RIGHT_ANGLE, Q2 3.1A/30V/105mΩ, U1 FSUSB30MUX_MSOP10, U2 AP63203, U3 ESD Diode, U5 ESD Diode, U6 CP210X

Commit message: Adds labels
Parts:
- C6: device SparkFun-Capacitors:10NF-0603-50V-10% -> SparkFun-Capacitors:10NF-0402T-25V-10%
- LOGO1: value SFE_LOGO_NAME_FLAME.1_INCH -> SFE_LOGO_NAME.1_INCH; device SparkFun-Aesthetics:SFE_LOGO_NAME_FLAME.1_INCH -> SparkFun-Aesthetics:SFE_LOGO_NAME.1_INCH
- LOGO3: value QWIIC_LOGO_3MM -> QWIIC_LOGO_5MM; device SparkFun-Aesthetics:QWIIC_LOGO_3MM -> SparkFun-Aesthetics:QWIIC_LOGO_5MM
- renumbered JP1 to PLED, JP3 to ALED
Changed lines of the file:
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@@
 <part name="SUPPLY15" library="SparkFun-PowerSymbols" deviceset="VIN" device=""/>
 <part name="SUPPLY9" library="SparkFun-PowerSymbols" deviceset="V_USB" device=""/>
-<part name="JP1" library="SparkFun-Jumpers" deviceset="JUMPER-SMT_2_NC_TRACE" device="_SILK" package3d_urn="urn:adsk.eagle:package:39281/1"/>
-<part name="JP3" library="SparkFun-Jumpers" deviceset="JUMPER-SMT_2_NC_TRACE" device="_SILK" package3d_urn="urn:adsk.eagle:package:39281/1"/>
-<part name="LOGO1" library="SparkFun-Aesthetics" deviceset="SFE_LOGO_NAME_FLAME" device=".1_INCH"/>
+<part name="PLED" library="SparkFun-Jumpers" deviceset="JUMPER-SMT_2_NC_TRACE" device="_SILK" package3d_urn="urn:adsk.eagle:package:39281/1"/>
+<part name="ALED" library="SparkFun-Jumpers" deviceset="JUMPER-SMT_2_NC_TRACE" device="_SILK" package3d_urn="urn:adsk.eagle:package:39281/1"/>
+<part name="LOGO1" library="SparkFun-Aesthetics" deviceset="SFE_LOGO_NAME" device=".1_INCH" value="SFE_LOGO_NAME.1_INCH"/>
 <part name="LOGO2" library="SparkFun-Aesthetics" deviceset="OSHW-LOGO" device="S"/>
-<part name="LOGO3" library="SparkFun-Aesthetics" deviceset="QWIIC_LOGO" device="_3MM"/>
+<part name="LOGO3" library="SparkFun-Aesthetics" deviceset="QWIIC_LOGO" device="_5MM" value="QWIIC_LOGO_5MM"/>
 <part name="U2" library="SparkFun-IC-Power" deviceset="AP63203" device="" value="AP63203"/>
 <part name="L1" library="SparkFun-Coils" deviceset="4.7μH_SHIELDED_INDUCTOR" device="NPIS_LS" value="4.7μH"/>
@@
 <part name="GND33" library="SparkFun-PowerSymbols" deviceset="GND" device=""/>
 <part name="GND34" library="SparkFun-PowerSymbols" deviceset="GND" device=""/>
-<part name="C6" library="SparkFun-Capacitors" deviceset="10NF" device="-0603-50V-10%" value="10nF"/>
+<part name="C6" library="SparkFun-Capacitors" deviceset="10NF" device="-0402T-25V-10%" value="10nF"/>
 <part name="GND7" library="SparkFun-PowerSymbols" deviceset="GND" device=""/>
 <part name="C7" library="SparkFun-Capacitors" deviceset="10NF" device="-0603-50V-10%" value="10nF"/>
@@
 <attribute name="VALUE" x="157.48" y="256.794" size="1.778" layer="96" font="vector" align="bottom-center"/>
 </instance>
-<instance part="JP1" gate="G$1" x="289.56" y="43.18" smashed="yes" rot="R90">
+<instance part="PLED" gate="G$1" x="289.56" y="43.18" smashed="yes" rot="R90">
 <attribute name="NAME" x="286.512" y="43.18" size="1.778" layer="95" font="vector" rot="R90" align="center"/>
 </instance>
-<instance part="JP3" gate="G$1" x="304.8" y="43.18" smashed="yes" rot="R90">
+<instance part="ALED" gate="G$1" x="304.8" y="43.18" smashed="yes" rot="R90">
 <attribute name="NAME" x="301.752" y="43.18" size="1.778" layer="95" font="vector" rot="R90" align="center"/>
 </instance>
@@
 </segment>
 <segment>
-<pinref part="JP3" gate="G$1" pin="1"/>
+<pinref part="ALED" gate="G$1" pin="1"/>
 <pinref part="GND14" gate="1" pin="GND"/>
 <wire x1="304.8" y1="38.1" x2="304.8" y2="35.56" width="0.1524" layer="91"/>
 </segment>
 <segment>
-<pinref part="JP1" gate="G$1" pin="1"/>
+<pinref part="PLED" gate="G$1" pin="1"/>
 <pinref part="GND12" gate="1" pin="GND"/>
 <wire x1="289.56" y1="38.1" x2="289.56" y2="35.56" width="0.1524" layer="91"/>
@@
 <net name="N$21" class="0">
 <segment>
-<pinref part="JP3" gate="G$1" pin="2"/>
+<pinref part="ALED" gate="G$1" pin="2"/>
 <pinref part="D3" gate="G$1" pin="C"/>
 <wire x1="304.8" y1="48.26" x2="304.8" y2="50.8" width="0.1524" layer="91"/>
@@
 <net name="N$23" class="0">
 <segment>
-<pinref part="JP1" gate="G$1" pin="2"/>
+<pinref part="PLED" gate="G$1" pin="2"/>
 <pinref part="D2" gate="G$1" pin="C"/>
 <wire x1="289.56" y1="48.26" x2="289.56" y2="50.8" width="0.1524" layer="91"/>

Commit message: Adds version
Parts:
- renumbered JP2 to J2
Other:
- note added: "v01"
- note removed: "v10"
Changed lines of the file:
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@@
 <part name="SUPPLY20" library="SparkFun-PowerSymbols" deviceset="V_USB_2" device=""/>
 <part name="GND31" library="SparkFun-PowerSymbols" deviceset="GND" device=""/>
-<part name="JP2" library="xbee_improved" deviceset="XBEE_UPDATE" device="XBEE_SMD"/>
+<part name="J2" library="xbee_improved" deviceset="XBEE_UPDATE" device="XBEE_SMD"/>
 <part name="U6" library="SparkFun-IC-Comms" deviceset="CP2102N" device="" value="CP210X"/>
 <part name="R9" library="SparkFun-Resistors" deviceset="10KOHM" device="-0603-1/10W-1%" value="10k"/>
@@
 <wire x1="294.64" y1="172.72" x2="431.8" y2="172.72" width="0.2032" layer="97" style="longdash"/>
 <wire x1="121.92" y1="111.76" x2="121.92" y2="0" width="0.2032" layer="97" style="longdash"/>
-<text x="424.18" y="7.62" size="2.54" layer="94" font="vector" align="center">v10</text>
+<text x="424.18" y="7.62" size="2.54" layer="94" font="vector" align="center">v01</text>
 <text x="363.22" y="10.16" size="2.54" layer="94" font="vector" align="center">Elias Santistevan</text>
 <text x="76.2" y="73.66" size="1.27" layer="97" font="vector">Default (Low) = SDA (I2C)</text>
@@
 <attribute name="VALUE" x="274.32" y="218.186" size="1.778" layer="96" font="vector" rot="MR0" align="top-center"/>
 </instance>
-<instance part="JP2" gate="G$1" x="60.96" y="218.44" smashed="yes">
+<instance part="J2" gate="G$1" x="60.96" y="218.44" smashed="yes">
 <attribute name="NAME" x="40.64" y="236.474" size="1.778" layer="95" font="vector"/>
 <attribute name="VALUE" x="40.64" y="200.406" size="1.778" layer="96" font="vector" align="top-left"/>
@@
 <wire x1="88.9" y1="226.06" x2="86.36" y2="226.06" width="0.1524" layer="91"/>
 <label x="88.9" y="226.06" size="1.27" layer="95" font="vector" rot="MR180" xref="yes"/>
-<pinref part="JP2" gate="G$1" pin="SCL/DIO1/AD1"/>
+<pinref part="J2" gate="G$1" pin="SCL/DIO1/AD1"/>
 </segment>
 <segment>
@@
 <wire x1="35.56" y1="200.66" x2="35.56" y2="203.2" width="0.1524" layer="91"/>
 <pinref part="GND22" gate="1" pin="GND"/>
-<pinref part="JP2" gate="G$1" pin="GND"/>
+<pinref part="J2" gate="G$1" pin="GND"/>
 </segment>
 <segment>
@@
 <wire x1="35.56" y1="236.22" x2="35.56" y2="233.68" width="0.1524" layer="91"/>
 <pinref part="SUPPLY10" gate="G$1" pin="3.3V"/>
-<pinref part="JP2" gate="G$1" pin="VCC"/>
+<pinref part="J2" gate="G$1" pin="VCC"/>
 <wire x1="35.56" y1="233.68" x2="38.1" y2="233.68" width="0.1524" layer="91"/>
 </segment>
@@
 <wire x1="35.56" y1="213.36" x2="38.1" y2="213.36" width="0.1524" layer="91"/>
 <label x="35.56" y="213.36" size="1.27" layer="95" font="vector" rot="MR0" xref="yes"/>
-<pinref part="JP2" gate="G$1" pin="DOUT"/>
+<pinref part="J2" gate="G$1" pin="DOUT"/>
 </segment>
 <segment>
@@
 <wire x1="35.56" y1="210.82" x2="38.1" y2="210.82" width="0.1524" layer="91"/>
 <label x="35.56" y="210.82" size="1.27" layer="95" font="vector" rot="MR0" xref="yes"/>
-<pinref part="JP2" gate="G$1" pin="DIN/!CONFIG!"/>
+<pinref part="J2" gate="G$1" pin="DIN/!CONFIG!"/>
 </segment>
 <segment>
@@
 <wire x1="88.9" y1="203.2" x2="86.36" y2="203.2" width="0.1524" layer="91"/>
 <label x="88.9" y="203.2" size="1.27" layer="95" font="vector" rot="MR180" xref="yes"/>
-<pinref part="JP2" gate="G$1" pin="POCI/DIO12"/>
+<pinref part="J2" gate="G$1" pin="POCI/DIO12"/>
 </segment>
 <segment>
@@
 <wire x1="111.76" y1="231.14" x2="109.22" y2="231.14" width="0.1524" layer="91"/>
 <label x="111.76" y="231.14" size="1.27" layer="95" font="vector" xref="yes"/>
-<pinref part="JP2" gate="G$1" pin="!RESET!"/>
+<pinref part="J2" gate="G$1" pin="!RESET!"/>
 <pinref part="C6" gate="G$1" pin="1"/>
 <wire x1="109.22" y1="231.14" x2="86.36" y2="231.14" width="0.1524" layer="91"/>
@@
 <wire x1="35.56" y1="228.6" x2="38.1" y2="228.6" width="0.1524" layer="91"/>
 <label x="35.56" y="228.6" size="1.27" layer="95" font="vector" rot="MR0" xref="yes"/>
-<pinref part="JP2" gate="G$1" pin="VUSB/RSSI/DIO10"/>
+<pinref part="J2" gate="G$1" pin="VUSB/RSSI/DIO10"/>
 </segment>
 <segment>
@@
 <wire x1="86.36" y1="208.28" x2="88.9" y2="208.28" width="0.1524" layer="91"/>
 <label x="88.9" y="208.28" size="1.27" layer="95" font="vector" rot="MR180" xref="yes"/>
-<pinref part="JP2" gate="G$1" pin="DTR/DIO8"/>
+<pinref part="J2" gate="G$1" pin="DTR/DIO8"/>
 </segment>
 <segment>
@@
 <wire x1="86.36" y1="218.44" x2="88.9" y2="218.44" width="0.1524" layer="91"/>
 <label x="88.9" y="218.44" size="1.27" layer="95" font="vector" rot="MR180" xref="yes"/>
-<pinref part="JP2" gate="G$1" pin="PICO/TX2/DIO4"/>
+<pinref part="J2" gate="G$1" pin="PICO/TX2/DIO4"/>
 </segment>
 <segment>
@@
 <wire x1="88.9" y1="210.82" x2="86.36" y2="210.82" width="0.1524" layer="91"/>
 <label x="88.9" y="210.82" size="1.27" layer="95" font="vector" rot="MR180" xref="yes"/>
-<pinref part="JP2" gate="G$1" pin="!CTS!/DIO7"/>
+<pinref part="J2" gate="G$1" pin="!CTS!/DIO7"/>
 </segment>
 <segment>
@@
 <wire x1="88.9" y1="205.74" x2="86.36" y2="205.74" width="0.1524" layer="91"/>
 <label x="88.9" y="205.74" size="1.27" layer="95" font="vector" rot="MR180" xref="yes"/>
-<pinref part="JP2" gate="G$1" pin="!SLEEP!/DIO9"/>
+<pinref part="J2" gate="G$1" pin="!SLEEP!/DIO9"/>
 </segment>
 <segment>
@@
 <wire x1="88.9" y1="215.9" x2="86.36" y2="215.9" width="0.1524" layer="91"/>
 <label x="88.9" y="215.9" size="1.27" layer="95" font="vector" rot="MR180" xref="yes"/>
-<pinref part="JP2" gate="G$1" pin="ASSOCIATE/DIO5"/>
+<pinref part="J2" gate="G$1" pin="ASSOCIATE/DIO5"/>
 </segment>
 <segment>
@@
 <wire x1="88.9" y1="213.36" x2="86.36" y2="213.36" width="0.1524" layer="91"/>
 <label x="88.9" y="213.36" size="1.27" layer="95" font="vector" rot="MR180" xref="yes"/>
-<pinref part="JP2" gate="G$1" pin="!RTS!/DIO6"/>
+<pinref part="J2" gate="G$1" pin="!RTS!/DIO6"/>
 </segment>
 <segment>
@@
 <wire x1="88.9" y1="220.98" x2="86.36" y2="220.98" width="0.1524" layer="91"/>
 <label x="88.9" y="220.98" size="1.27" layer="95" font="vector" rot="MR180" xref="yes"/>
-<pinref part="JP2" gate="G$1" pin="!CS!/!CTS2!/DIO3/AD3"/>
+<pinref part="J2" gate="G$1" pin="!CS!/!CTS2!/DIO3/AD3"/>
 </segment>
 <segment>
@@
 <wire x1="88.9" y1="223.52" x2="86.36" y2="223.52" width="0.1524" layer="91"/>
 <label x="88.9" y="223.52" size="1.27" layer="95" font="vector" rot="MR180" xref="yes"/>
-<pinref part="JP2" gate="G$1" pin="ATTN/CLK/!RTS2!/DIO2/AD2"/>
+<pinref part="J2" gate="G$1" pin="ATTN/CLK/!RTS2!/DIO2/AD2"/>
 </segment>
 <segment>
@@
 <wire x1="88.9" y1="228.6" x2="86.36" y2="228.6" width="0.1524" layer="91"/>
 <label x="88.9" y="228.6" size="1.27" layer="95" font="vector" rot="MR180" xref="yes"/>
-<pinref part="JP2" gate="G$1" pin="DIO0/AD0"/>
+<pinref part="J2" gate="G$1" pin="DIO0/AD0"/>
 </segment>
 </net>
@@
 <wire x1="35.56" y1="226.06" x2="38.1" y2="226.06" width="0.1524" layer="91"/>
 <label x="35.56" y="226.06" size="1.27" layer="95" font="vector" rot="R180" xref="yes"/>
-<pinref part="JP2" gate="G$1" pin="D+/SDA/DIO11"/>
+<pinref part="J2" gate="G$1" pin="D+/SDA/DIO11"/>
 </segment>
 <segment>
@@
 <wire x1="35.56" y1="223.52" x2="38.1" y2="223.52" width="0.1524" layer="91"/>
 <label x="35.56" y="223.52" size="1.27" layer="95" font="vector" rot="R180" xref="yes"/>
-<pinref part="JP2" gate="G$1" pin="D-"/>
-</segment>
-<segment>
+<pinref part="J2" gate="G$1" pin="D-"/>
+</segment>
+<segment>
