File: Hardware/SparkFun_XBee_Development_Board.brd (EAGLE design)
At the start: 45.7 x 63.5 mm, 138 parts, among them J1 USB Female Type C Connector, J3 USB Female Type C Connector, J4 QWIIC_RIGHT_ANGLE, Q2 3.1A/30V/105mΩ, U1 FSUSB30MUX_MSOP10, U2 AP63203, U3 ESD Diode, U5 ESD Diode, U7 FT231XS

Commit message: Adds production files, shifts buttons down just a bit
Parts:
- moved S1 1.27 mm to (3.17, 41.9)
- moved S2 1.27 mm to (42.5, 41.9)
- moved LOGO2 0.64 mm to (42.5, 49.5)
- moved U$30 0.38 mm to (3.43, 46.5)
- moved U$40 0.38 mm to (42.5, 46.5)
Routing:
- net D0: track 15.7 -> 14.0 mm
- net !RESET!: track 19.7 -> 18.6 mm
- net GND: vias 82 -> 85
